Commit message: 1、fix meshes path error  2,update readme

File: star1/urdf/l3_with_hand_fixedpin_xml.urdf (robot description, URDF)
Before this commit: robot l3, 80 links, 79 joints
Links:
- link base_link: geometry collision mesh filename=../meshes/base_link.STL; visual mesh filename=../meshes/base_link.STL
- link base_rs_link: geometry collision mesh filename=../meshes/base_rs_link.STL; visual mesh filename=../meshes/base_rs_link.STL
- link head_rs_link: geometry collision mesh filename=../meshes/head_rs_link.STL; visual mesh filename=../meshes/head_rs_link.STL
- link left_ankle_pitch_link: geometry collision mesh filename=../meshes/left_ankle_pitch_link.STL; visual mesh filename=../meshes/left_ankle_pitch_link.STL
- link left_ankle_roll_link: geometry collision mesh filename=../meshes/left_ankle_roll_link.STL; visual mesh filename=../meshes/left_ankle_roll_link.STL
- link left_arm_base_link: geometry collision mesh filename=../meshes/left_arm_base_link.STL; visual mesh filename=../meshes/left_arm_base_link.STL
- link left_arm_yaw_link: geometry collision mesh filename=../meshes/left_arm_yaw_link.STL; visual mesh filename=../meshes/left_arm_yaw_link.STL
- link left_elbow_pitch_link: geometry collision mesh filename=../meshes/left_elbow_pitch_link.STL; visual mesh filename=../meshes/left_elbow_pitch_link.STL
- link left_elbow_yaw_link: geometry collision mesh filename=../meshes/left_elbow_yaw_link.STL; visual mesh filename=../meshes/left_elbow_yaw_link.STL
- link left_hand_base_link: geometry collision mesh filename=../meshes/left_hand_base_link.STL; visual mesh filename=../meshes/left_hand_base_link.STL
- link left_hand_ee_link: geometry collision mesh filename=../meshes/left_hand_ee_link.STL; visual mesh filename=../meshes/left_hand_ee_link.STL
- link left_hand_index_bend_link: geometry collision mesh filename=../meshes/left_hand_index_bend_link.STL; visual mesh filename=../meshes/left_hand_index_bend_link.STL
- link left_hand_index_rota_link1: geometry collision mesh filename=../meshes/left_hand_index_rota_link1.STL; visual mesh filename=../meshes/left_hand_index_rota_link1.STL
- link left_hand_index_rota_link2: geometry collision mesh filename=../meshes/left_hand_index_rota_link2.STL; visual mesh filename=../meshes/left_hand_index_rota_link2.STL
- link left_hand_index_rota_tip: geometry collision mesh filename=../meshes/left_hand_index_rota_tip.STL; visual mesh filename=../meshes/left_hand_index_rota_tip.STL
- link left_hand_link: geometry collision mesh filename=../meshes/left_hand_link.STL; visual mesh filename=../meshes/left_hand_link.STL
- link left_hand_mid_link1: geometry collision mesh filename=../meshes/left_hand_mid_link1.STL; visual mesh filename=../meshes/left_hand_mid_link1.STL
- link left_hand_mid_link2: geometry collision mesh filename=../meshes/left_hand_mid_link2.STL; visual mesh filename=../meshes/left_hand_mid_link2.STL
- link left_hand_mid_tip: geometry collision mesh filename=../meshes/left_hand_mid_tip.STL; visual mesh filename=../meshes/left_hand_mid_tip.STL
- link left_hand_pinky_link1: geometry collision mesh filename=../meshes/left_hand_pinky_link1.STL; visual mesh filename=../meshes/left_hand_pinky_link1.STL
- link left_hand_pinky_link2: geometry collision mesh filename=../meshes/left_hand_pinky_link2.STL; visual mesh filename=../meshes/left_hand_pinky_link2.STL
- link left_hand_pinky_tip: geometry collision mesh filename=../meshes/left_hand_pinky_tip.STL; visual mesh filename=../meshes/left_hand_pinky_tip.STL
- link left_hand_ring_link1: geometry collision mesh filename=../meshes/left_hand_ring_link1.STL; visual mesh filename=../meshes/left_hand_ring_link1.STL
- link left_hand_ring_link2: geometry collision mesh filename=../meshes/left_hand_ring_link2.STL; visual mesh filename=../meshes/left_hand_ring_link2.STL
- link left_hand_ring_tip: geometry collision mesh filename=../meshes/left_hand_ring_tip.STL; visual mesh filename=../meshes/left_hand_ring_tip.STL
- link left_hand_thumb_bend_link: geometry collision mesh filename=../meshes/left_hand_thumb_bend_link.STL; visual mesh filename=../meshes/left_hand_thumb_bend_link.STL
- link left_hand_thumb_rota_link1: geometry collision mesh filename=../meshes/left_hand_thumb_rota_link1.STL; visual mesh filename=../meshes/left_hand_thumb_rota_link1.STL
- link left_hand_thumb_rota_link2: geometry collision mesh filename=../meshes/left_hand_thumb_rota_link2.STL; visual mesh filename=../meshes/left_hand_thumb_rota_link2.STL
- link left_hand_thumb_rota_tip: geometry collision mesh filename=../meshes/left_hand_thumb_rota_tip.STL; visual mesh filename=../meshes/left_hand_thumb_rota_tip.STL
- link left_hip_pitch_link: geometry collision mesh filename=../meshes/left_hip_pitch_link.STL; visual mesh filename=../meshes/left_hip_pitch_link.STL
- link left_hip_roll_link: geometry collision mesh filename=../meshes/left_hip_roll_link.STL; visual mesh filename=../meshes/left_hip_roll_link.STL
- link left_hip_yaw_link: geometry collision mesh filename=../meshes/left_hip_yaw_link.STL; visual mesh filename=../meshes/left_hip_yaw_link.STL
- link left_knee_link: geometry collision mesh filename=../meshes/left_knee_link.STL; visual mesh filename=../meshes/left_knee_link.STL
- link left_shoulder_pitch_link: geometry collision mesh filename=../meshes/left_shoulder_pitch_link.STL; visual mesh filename=../meshes/left_shoulder_pitch_link.STL
- link left_shoulder_roll_link: geometry collision mesh filename=../meshes/left_shoulder_roll_link.STL; visual mesh filename=../meshes/left_shoulder_roll_link.STL
- link left_wrist_pitch_link: geometry collision mesh filename=../meshes/left_wrist_pitch_link.STL; visual mesh filename=../meshes/left_wrist_pitch_link.STL
- link left_wrist_roll_link: geometry collision mesh filename=../meshes/left_wrist_roll_link.STL; visual mesh filename=../meshes/left_wrist_roll_link.STL
- link mic_link: geometry collision mesh filename=../meshes/mic_link.STL; visual mesh filename=../meshes/mic_link.STL
- link neck_pitch_link: geometry collision mesh filename=../meshes/neck_pitch_link.STL; visual mesh filename=../meshes/neck_pitch_link.STL
- link neck_yaw_link: geometry collision mesh filename=../meshes/neck_yaw_link.STL; visual mesh filename=../meshes/neck_yaw_link.STL
- link right_ankle_pitch_link: geometry collision mesh filename=../meshes/right_ankle_pitch_link.STL; visual mesh filename=../meshes/right_ankle_pitch_link.STL
- link right_ankle_roll_link: geometry collision mesh filename=../meshes/right_ankle_roll_link.STL; visual mesh filename=../meshes/right_ankle_roll_link.STL
- link right_arm_base_link: geometry collision mesh filename=../meshes/right_arm_base_link.STL; visual mesh filename=../meshes/right_arm_base_link.STL
- link right_arm_yaw_link: geometry collision mesh filename=../meshes/right_arm_yaw_link.STL; visual mesh filename=../meshes/right_arm_yaw_link.STL
- link right_elbow_pitch_link: geometry collision mesh filename=../meshes/right_elbow_pitch_link.STL; visual mesh filename=../meshes/right_elbow_pitch_link.STL
- link right_elbow_yaw_link: geometry collision mesh filename=../meshes/right_elbow_yaw_link.STL; visual mesh filename=../meshes/right_elbow_yaw_link.STL
- link right_hand_base_link: geometry collision mesh filename=../meshes/right_hand_base_link.STL; visual mesh filename=../meshes/right_hand_base_link.STL
- link right_hand_ee_link: geometry collision mesh filename=../meshes/right_hand_ee_link.STL; visual mesh filename=../meshes/right_hand_ee_link.STL
- link right_hand_index_bend_link: geometry collision mesh filename=../meshes/right_hand_index_bend_link.STL; visual mesh filename=../meshes/right_hand_index_bend_link.STL
- link right_hand_index_rota_link1: geometry collision mesh filename=../meshes/right_hand_index_rota_link1.STL; visual mesh filename=../meshes/right_hand_index_rota_link1.STL
- link right_hand_index_rota_link2: geometry collision mesh filename=../meshes/right_hand_index_rota_link2.STL; visual mesh filename=../meshes/right_hand_index_rota_link2.STL
- link right_hand_index_rota_tip: geometry collision mesh filename=../meshes/right_hand_index_rota_tip.STL; visual mesh filename=../meshes/right_hand_index_rota_tip.STL
- link right_hand_link: geometry collision mesh filename=../meshes/right_hand_link.STL; visual mesh filename=../meshes/right_hand_link.STL
- link right_hand_mid_link1: geometry collision mesh filename=../meshes/right_hand_mid_link1.STL; visual mesh filename=../meshes/right_hand_mid_link1.STL
- link right_hand_mid_link2: geometry collision mesh filename=../meshes/right_hand_mid_link2.STL; visual mesh filename=../meshes/right_hand_mid_link2.STL
- link right_hand_mid_tip: geometry collision mesh filename=../meshes/right_hand_mid_tip.STL; visual mesh filename=../meshes/right_hand_mid_tip.STL
- link right_hand_pinky_link1: geometry collision mesh filename=../meshes/right_hand_pinky_link1.STL; visual mesh filename=../meshes/right_hand_pinky_link1.STL
- link right_hand_pinky_link2: geometry collision mesh filename=../meshes/right_hand_pinky_link2.STL; visual mesh filename=../meshes/right_hand_pinky_link2.STL
- link right_hand_pinky_tip: geometry collision mesh filename=../meshes/right_hand_pinky_tip.STL; visual mesh filename=../meshes/right_hand_pinky_tip.STL
- link right_hand_ring_link1: geometry collision mesh filename=../meshes/right_hand_ring_link1.STL; visual mesh filename=../meshes/right_hand_ring_link1.STL
- link right_hand_ring_link2: geometry collision mesh filename=../meshes/right_hand_ring_link2.STL; visual mesh filename=../meshes/right_hand_ring_link2.STL
- link right_hand_ring_tip: geometry collision mesh filename=../meshes/right_hand_ring_tip.STL; visual mesh filename=../meshes/right_hand_ring_tip.STL
- link right_hand_thumb_bend_link: geometry collision mesh filename=../meshes/right_hand_thumb_bend_link.STL; visual mesh filename=../meshes/right_hand_thumb_bend_link.STL
- link right_hand_thumb_rota_link1: geometry collision mesh filename=../meshes/right_hand_thumb_rota_link1.STL; visual mesh filename=../meshes/right_hand_thumb_rota_link1.STL
- link right_hand_thumb_rota_link2: geometry collision mesh filename=../meshes/right_hand_thumb_rota_link2.STL; visual mesh filename=../meshes/right_hand_thumb_rota_link2.STL
- link right_hand_thumb_rota_tip: geometry collision mesh filename=../meshes/right_hand_thumb_rota_tip.STL; visual mesh filename=../meshes/right_hand_thumb_rota_tip.STL
- link right_hip_pitch_link: geometry collision mesh filename=../meshes/right_hip_pitch_link.STL; visual mesh filename=../meshes/right_hip_pitch_link.STL
- link right_hip_roll_link: geometry collision mesh filename=../meshes/right_hip_roll_link.STL; visual mesh filename=../meshes/right_hip_roll_link.STL
- link right_hip_yaw_link: geometry collision mesh filename=../meshes/right_hip_yaw_link.STL; visual mesh filename=../meshes/right_hip_yaw_link.STL
- link right_knee_link: geometry collision mesh filename=../meshes/right_knee_link.STL; visual mesh filename=../meshes/right_knee_link.STL
- link right_shoulder_pitch_link: geometry collision mesh filename=../meshes/right_shoulder_pitch_link.STL; visual mesh filename=../meshes/right_shoulder_pitch_link.STL
- link right_shoulder_roll_link: geometry collision mesh filename=../meshes/right_shoulder_roll_link.STL; visual mesh filename=../meshes/right_shoulder_roll_link.STL
- link right_wrist_pitch_link: geometry collision mesh filename=../meshes/right_wrist_pitch_link.STL; visual mesh filename=../meshes/right_wrist_pitch_link.STL
- link right_wrist_roll_link: geometry collision mesh filename=../meshes/right_wrist_roll_link.STL; visual mesh filename=../meshes/right_wrist_roll_link.STL
- link waist_base_link: geometry collision mesh filename=../meshes/waist_base_link.STL; visual mesh filename=../meshes/waist_base_link.STL
- link waist_pitch_link: geometry collision mesh filename=../meshes/waist_pitch_link.STL; visual mesh filename=../meshes/waist_pitch_link.STL
- link waist_roll_link: geometry collision mesh filename=../meshes/waist_roll_link.STL; visual mesh filename=../meshes/waist_roll_link.STL
- link waist_yaw_link: geometry collision mesh filename=../meshes/waist_yaw_link.STL; visual mesh filename=../meshes/waist_yaw_link.STL

Commit message: rm realsense

File: star1/urdf/l3_with_hand_fixedpin_xml.urdf (robot description, URDF)
Before this commit: robot l3, 80 links, 79 joints
Links:
- removed link base_rs_link
Joints:
- removed joint base_rs_joint
